File: nindo.kicad_sch (KiCad schematic)
At the start: 64 parts, among them J1 Micro_SD_Card_Det1, J2 USB_C_Receptacle_USB2.0_16P, J3 Conn_01x08_Pin, J4 AudioJack3, SW1 SW_MEC_5G, SW2 SW_MEC_5G, SW3 SW_MEC_5G, SW4 SW_MEC_5G, SW5 SW_MEC_5G, SW6 SW_MEC_5G, SW7 SW_MEC_5G, SW8 SW_MEC_5G, SW9 SW_MEC_5G, U1 PCM5102A, U2 ESP32-S3-WROOM-1, U3 TP4056-42-ESOP8, U4 DW01A, U5 ME6211C33M5

Commit message: hhhh
Parts:
- added J5: Conn_01x02_Pin, Connector:JWT_A3963_1x02_P3.96mm_Vertical, symbol Connector:Conn_01x02_Pin
- C1, C10, C11, C12, C13, C14, C15, C16, C17, C2, C20, C3, C4, C5, C6, C7, C8, C9: footprint (none) -> Capacitor_SMD:C_1206_3216Metric_Pad1.33x1.80mm_HandSolder
- R1, R10, R11, R12, R13, R14, R15, R16, R17, R18, R19, R2, R20, R21, R22, R23, R24, R25, R26, R27, R3, R4, R5, R6, R7, R8, R9: footprint (none) -> Resistor_SMD:R_1206_3216Metric_Pad1.30x1.75mm_HandSolder
Connections:
- net B+: now also J5.1 (Pin_1)
- net B-: now also J5.2 (Pin_2)
