File: nindo.kicad_pcb (KiCad board)
At the start: 2 copper layers, 4 parts, among them U1 PCM5102A, U2 ESP32-S3-WROOM-1, U3 TP4056-42-ESOP8, U4 DW01A

Commit message: hhhh
Parts:
- added 8205A1: ~, Package_TO_SOT_SMD:SOT-23-6, B.Cu at (122.6, 112.5)
- added C1: 0.1u, Capacitor_SMD:C_1206_3216Metric_Pad1.33x1.80mm_HandSolder, B.Cu at (123.0, 92.0)
- added C10: 10u, Capacitor_SMD:C_1206_3216Metric_Pad1.33x1.80mm_HandSolder, F.Cu at (128.1, 75.0)
- added C11: 10u, Capacitor_SMD:C_1206_3216Metric_Pad1.33x1.80mm_HandSolder, F.Cu at (172.5, 77.5)
- added C12: 10u, Capacitor_SMD:C_1206_3216Metric_Pad1.33x1.80mm_HandSolder, B.Cu at (155.0, 100.0)
- added C13: 1u, Capacitor_SMD:C_1206_3216Metric_Pad1.33x1.80mm_HandSolder, B.Cu at (153.5, 110.0)
- added C14: 100n, Capacitor_SMD:C_1206_3216Metric_Pad1.33x1.80mm_HandSolder, B.Cu at (148.0, 96.5)
- added C15: 100n, Capacitor_SMD:C_1206_3216Metric_Pad1.33x1.80mm_HandSolder, B.Cu at (139.5, 108.0)
- added C16: 100n, Capacitor_SMD:C_1206_3216Metric_Pad1.33x1.80mm_HandSolder, B.Cu at (148.5, 112.0)
- added C17: 10u, Capacitor_SMD:C_1206_3216Metric_Pad1.33x1.80mm_HandSolder, B.Cu at (146.0, 112.0)
- added C2: 0.1u, Capacitor_SMD:C_1206_3216Metric_Pad1.33x1.80mm_HandSolder, B.Cu at (111.5, 107.5)
- added C20: 100n, Capacitor_SMD:C_1206_3216Metric_Pad1.33x1.80mm_HandSolder, B.Cu at (155.0, 105.5)
- added C3: 10u, Capacitor_SMD:C_1206_3216Metric_Pad1.33x1.80mm_HandSolder, B.Cu at (109.0, 97.0)
- added C4: 10u, Capacitor_SMD:C_1206_3216Metric_Pad1.33x1.80mm_HandSolder, B.Cu at (116.5, 114.0)
- added C5: 10u, Capacitor_SMD:C_1206_3216Metric_Pad1.33x1.80mm_HandSolder, B.Cu at (116.5, 111.0)
- added C6: 100n, Capacitor_SMD:C_1206_3216Metric_Pad1.33x1.80mm_HandSolder, F.Cu at (128.1, 72.5)
- added C7: 100n, Capacitor_SMD:C_1206_3216Metric_Pad1.33x1.80mm_HandSolder, F.Cu at (172.5, 72.5)
- added C8: 100n, Capacitor_SMD:C_1206_3216Metric_Pad1.33x1.80mm_HandSolder, F.Cu at (128.1, 67.5)
- added C9: 10u, Capacitor_SMD:C_1206_3216Metric_Pad1.33x1.80mm_HandSolder, F.Cu at (128.1, 70.0)
- added J1: Micro_SD_Card_Det1, Connector_Card:microSD_HC_Hirose_DM3AT-SF-PEJM5, B.Cu at (177.5, 76.0)
- added J2: USB_C_Receptacle_USB2.0_16P, Connector_USB:USB_C_Receptacle_G-Switch_GT-USB-7010ASV, F.Cu at (183.5, 107.5)
- added J3: Conn_01x08_Pin, Connector_Harwin:Harwin_M20-89008xx_1x08_P2.54mm_Horizontal, B.Cu at (95.5, 78.9)
- added J4: AudioJack3, Connector_Audio:Jack_3.5mm_CUI_SJ1-3523N_Horizontal, F.Cu at (182.5, 94.0)
- added J5: Conn_01x02_Pin, Connector:JWT_A3963_1x02_P3.96mm_Vertical, F.Cu at (98.1, 97.1)
- added R1: 1K2, Resistor_SMD:R_1206_3216Metric_Pad1.30x1.75mm_HandSolder, B.Cu at (115.0, 98.5)
- added R10: 10k, Resistor_SMD:R_1206_3216Metric_Pad1.30x1.75mm_HandSolder, B.Cu at (134.5, 119.0)
- added R11: 10k, Resistor_SMD:R_1206_3216Metric_Pad1.30x1.75mm_HandSolder, B.Cu at (133.5, 131.0)
- added R12: 10k, Resistor_SMD:R_1206_3216Metric_Pad1.30x1.75mm_HandSolder, B.Cu at (117.5, 129.0)
- added R13: 10k, Resistor_SMD:R_1206_3216Metric_Pad1.30x1.75mm_HandSolder, B.Cu at (151.0, 129.0)
- added R14: 10k, Resistor_SMD:R_1206_3216Metric_Pad1.30x1.75mm_HandSolder, B.Cu at (174.5, 121.0)
- added R15: 10k, Resistor_SMD:R_1206_3216Metric_Pad1.30x1.75mm_HandSolder, B.Cu at (174.0, 131.0)
- added R16: 10k, Resistor_SMD:R_1206_3216Metric_Pad1.30x1.75mm_HandSolder, B.Cu at (101.0, 129.0)
- added R17: 10k, Resistor_SMD:R_1206_3216Metric_Pad1.30x1.75mm_HandSolder, B.Cu at (102.0, 110.0)
- added R18: 10k, Resistor_SMD:R_1206_3216Metric_Pad1.30x1.75mm_HandSolder, B.Cu at (115.0, 79.5)
- added R19: 33, Resistor_SMD:R_1206_3216Metric_Pad1.30x1.75mm_HandSolder, B.Cu at (115.0, 83.5)
- added R2: 5K1, Resistor_SMD:R_1206_3216Metric_Pad1.30x1.75mm_HandSolder, F.Cu at (167.5, 108.5)
- added R20: 100k, Resistor_SMD:R_1206_3216Metric_Pad1.30x1.75mm_HandSolder, B.Cu at (156.0, 95.0)
- added R21: 100k, Resistor_SMD:R_1206_3216Metric_Pad1.30x1.75mm_HandSolder, B.Cu at (138.5, 100.0)
- added R22: 100, Resistor_SMD:R_1206_3216Metric_Pad1.30x1.75mm_HandSolder, B.Cu at (167.5, 90.5)
- added R23: 100, Resistor_SMD:R_1206_3216Metric_Pad1.30x1.75mm_HandSolder, B.Cu at (167.5, 97.0)
- added R24: 10k, Resistor_SMD:R_1206_3216Metric_Pad1.30x1.75mm_HandSolder, B.Cu at (164.0, 73.5)
- added R25: 10k, Resistor_SMD:R_1206_3216Metric_Pad1.30x1.75mm_HandSolder, B.Cu at (164.0, 76.5)
- added R26: 10k, Resistor_SMD:R_1206_3216Metric_Pad1.30x1.75mm_HandSolder, B.Cu at (163.0, 80.5)
- added R27: 10k, Resistor_SMD:R_1206_3216Metric_Pad1.30x1.75mm_HandSolder, B.Cu at (164.0, 70.0)
- added R3: 5K1, Resistor_SMD:R_1206_3216Metric_Pad1.30x1.75mm_HandSolder, F.Cu at (167.5, 105.0)
- added R4: 1k, Resistor_SMD:R_1206_3216Metric_Pad1.30x1.75mm_HandSolder, B.Cu at (127.0, 107.5)
- added R5: 100, Resistor_SMD:R_1206_3216Metric_Pad1.30x1.75mm_HandSolder, B.Cu at (110.5, 103.0)
- added R6: 10k, Resistor_SMD:R_1206_3216Metric_Pad1.30x1.75mm_HandSolder, B.Cu at (125.5, 98.5)
- added R7: 10k, Resistor_SMD:R_1206_3216Metric_Pad1.30x1.75mm_HandSolder, B.Cu at (142.1, 68.0)
- added R8: 10k, Resistor_SMD:R_1206_3216Metric_Pad1.30x1.75mm_HandSolder, B.Cu at (163.0, 83.0)
- added R9: 10k, Resistor_SMD:R_1206_3216Metric_Pad1.30x1.75mm_HandSolder, B.Cu at (164.0, 67.5)
- added SW1: SW_MEC_5G, Button_Switch_SMD:SW_MEC_5GSH9, F.Cu at (134.5, 121.5)
- added SW2: SW_MEC_5G, Button_Switch_SMD:SW_MEC_5GSH9, F.Cu at (134.5, 134.0)
- added SW3: SW_MEC_5G, Button_Switch_SMD:SW_MEC_5GSH9, F.Cu at (116.5, 129.0)
- added SW4: SW_MEC_5G, Button_Switch_SMD:SW_MEC_5GSH9, F.Cu at (152.0, 129.0)
- added SW5: SW_MEC_5G, Button_Switch_SMD:SW_MEC_5GSH9, F.Cu at (174.5, 120.5)
- added SW6: SW_MEC_5G, Button_Switch_SMD:SW_MEC_5GSH9, F.Cu at (174.5, 131.5)
- added SW7: SW_MEC_5G, Button_Switch_SMD:SW_MEC_5GSH9, F.Cu at (101.0, 128.5)
- added SW8: SW_MEC_5G, Button_Switch_SMD:SW_MEC_5GSH9, F.Cu at (101.0, 109.0)
- added SW9: SW_MEC_5G, Button_Switch_SMD:SW_MEC_5GSH9, F.Cu at (115.0, 80.5)
- added U5: ME6211C33M5, Package_TO_SOT_SMD:SOT-23-5, B.Cu at (117.0, 106.3)
- U1, U3, U4: moved to B.Cu
- moved U1 80.1 mm to (147.9, 102.9), turned to 90 degrees
- moved U4 46.0 mm to (122.5, 104.5), turned to 180 degrees
- moved U3 44.9 mm to (119.9, 97.0), turned to 90 degrees
- moved U2 12.1 mm to (147.1, 71.8)
Connections:
- U1 pad 1: unconnected-(U1-CPVDD-Pad1) -> +3.3V
- U1 pad 10: unconnected-(U1-DEMP-Pad10) -> GND
- U1 pad 11: unconnected-(U1-FLT-Pad11) -> GND
- U1 pad 12: unconnected-(U1-SCK-Pad12) -> Net-(U1-SCK)
- U1 pad 13: unconnected-(U1-BCK-Pad13) -> BCK_AUD
- U1 pad 14: unconnected-(U1-DIN-Pad14) -> DIN_AUD
- U1 pad 15: unconnected-(U1-LRCK-Pad15) -> LRCK_AUD
- U1 pad 16: unconnected-(U1-FMT-Pad16) -> GND
- U1 pad 17: unconnected-(U1-XSMT-Pad17) -> Net-(U1-XSMT)
- U1 pad 18: unconnected-(U1-LDOO-Pad18) -> Net-(U1-LDOO)
- U1 pad 19: unconnected-(U1-DGND-Pad19) -> GND
- U1 pad 2: unconnected-(U1-CAPP-Pad2) -> Net-(U1-CAPP)
- U1 pad 20: unconnected-(U1-DVDD-Pad20) -> +3.3V
- U1 pad 3: unconnected-(U1-CPGND-Pad3) -> GND
- U1 pad 4: unconnected-(U1-CAPM-Pad4) -> Net-(U1-CAPM)
- U1 pad 5: unconnected-(U1-VNEG-Pad5) -> Net-(U1-VNEG)
- U1 pad 6: unconnected-(U1-OUTL-Pad6) -> Net-(U1-OUTL)
- U1 pad 7: unconnected-(U1-OUTR-Pad7) -> Net-(U1-OUTR)
- U1 pad 8: unconnected-(U1-AVDD-Pad8) -> +3.3V
- U1 pad 9: unconnected-(U1-AGND-Pad9) -> GND
- U2 pad 1: Net-(U2-GND-Pad1) -> GND
- U2 pad 10: unconnected-(U2-IO17-Pad10) -> B_B
- U2 pad 11: unconnected-(U2-IO18-Pad11) -> S7AR7_B
- U2 pad 12: unconnected-(U2-IO8-Pad12) -> LEF_B
- U2 pad 13: unconnected-(U2-USB_D--Pad13) -> D-
- U2 pad 14: unconnected-(U2-USB_D+-Pad14) -> D+
- U2 pad 17: unconnected-(U2-IO9-Pad17) -> RIGH_B
- U2 pad 18: unconnected-(U2-IO10-Pad18) -> CS_DISP
- U2 pad 19: unconnected-(U2-IO11-Pad19) -> DIN_DISP
- U2 pad 2: unconnected-(U2-3V3-Pad2) -> +3.3V
- U2 pad 20: unconnected-(U2-IO12-Pad20) -> CLK_DISP
- U2 pad 21: unconnected-(U2-IO13-Pad21) -> DC_DISP
- U2 pad 22: unconnected-(U2-IO14-Pad22) -> RST_DISP
- U2 pad 23: unconnected-(U2-IO21-Pad23) -> CS_SDC
- U2 pad 27: unconnected-(U2-IO0-Pad27) -> BOO7_B
- U2 pad 3: unconnected-(U2-EN-Pad3) -> Net-(U2-EN)
- U2 pad 31: unconnected-(U2-IO38-Pad31) -> DE7_SDC
- U2 pad 33: unconnected-(U2-IO40-Pad33) -> MOSI_SDC
- U2 pad 34: unconnected-(U2-IO41-Pad34) -> MISO_SDC
- U2 pad 35: unconnected-(U2-IO42-Pad35) -> CLK_SDC
- U2 pad 38: unconnected-(U2-IO2-Pad38) -> DOWN_B
- U2 pad 39: unconnected-(U2-IO1-Pad39) -> UP_B
- U2 pad 4: unconnected-(U2-IO4-Pad4) -> SELEC_B
- U2 pad 40: Net-(U2-GND-Pad1) -> GND
- U2 pad 41: Net-(U2-GND-Pad1) -> GND
- U2 pad 5: unconnected-(U2-IO5-Pad5) -> LRCK_AUD
- U2 pad 6: unconnected-(U2-IO6-Pad6) -> BCK_AUD
- U2 pad 7: unconnected-(U2-IO7-Pad7) -> DIN_AUD
- U2 pad 8: unconnected-(U2-IO15-Pad8) -> BL_DISP
- U2 pad 9: unconnected-(U2-IO16-Pad9) -> A_B
- U3 pad 1: unconnected-(U3-TEMP-Pad1) -> Net-(U3-TEMP)
- U3 pad 2: unconnected-(U3-PROG-Pad2) -> Net-(U3-PROG)
- U3 pad 3: unconnected-(U3-GND-Pad3) -> GND
- U3 pad 4: unconnected-(U3-V_{CC}-Pad4) -> +5V
- U3 pad 5: unconnected-(U3-BAT-Pad5) -> B+
- U3 pad 8: unconnected-(U3-CE-Pad8) -> +5V
- U4 pad 1: unconnected-(U4-OD-Pad1) -> Net-(8205A1-G2)
- U4 pad 2: unconnected-(U4-CS-Pad2) -> Net-(U4-CS)
- U4 pad 3: unconnected-(U4-OC-Pad3) -> Net-(8205A1-G1)
- U4 pad 5: unconnected-(U4-VCC-Pad5) -> Net-(U4-VCC)
- U4 pad 6: unconnected-(U4-GND-Pad6) -> B-
Routing:
- net GND: track 0.00 -> 20.9 mm
- net Net-(J4-PadR): track 0.00 -> 9.28 mm
- net Net-(J4-PadT): track 0.00 -> 9.07 mm
- net +3.3V: track 0.00 -> 7.20 mm, vias 0 -> 1
- net Net-(U2-EN): track 0.00 -> 3.98 mm, vias 0 -> 1
Other:
- board outline added: 93.5 x 75.5 mm

Commit message: pcb
Routing:
- net RIGH_B: track 0.00 -> 65.6 mm, vias 0 -> 2
- net +3.3V: track 7.20 -> 71.0 mm, vias 1 -> 6
- net DC_DISP: track 0.00 -> 63.7 mm, vias 0 -> 5
- net RST_DISP: track 0.00 -> 60.8 mm, vias 0 -> 1
- net DIN_DISP: track 0.00 -> 58.9 mm, vias 0 -> 3
- net CLK_DISP: track 0.00 -> 50.8 mm, vias 0 -> 3
- net CS_DISP: track 0.00 -> 44.0 mm, vias 0 -> 1
- net GND: track 20.9 -> 61.2 mm, vias 0 -> 5
- net CS_SDC: track 0.00 -> 23.8 mm, vias 0 -> 3
- net B_B: track 0.00 -> 19.0 mm, vias 0 -> 4
- net Net-(J1-DAT2): track 0.00 -> 8.46 mm, vias 0 -> 2
